File: kicad-hamster-esp8266.kicad_pcb (KiCad board)
At the start: 2 copper layers, 85 x 51 mm, 32 parts, among them J1 Power Supply, J2 UART, J3 Screw_Terminal_01x08, Q1 IRLML5203, SW1 Reset, SW2 Flash, U1 ADM706P, U2 MC34063AD, U3 ESP-12F, U4 LM75B

Commit message: update legend and gerbers
- add reed switch connector legend
- regenerate gerbers

Signed-off-by: Sergey Matyukevich <geomatsi@gmail.com>
Other:
- board text added: "12"
- board text added: "13"
- board text added: "14"
- board text added: "16"
